File: hardware/dropdown/dropdown.kicad_sch (KiCad schematic)
At the start: 14 parts, among them J1 12, J1 3, J1 G, J1 T1, J1 T2, U1 AP7381-33Y-13

Commit message: feat: 4 layers PCB + AMS1117 (#17)
* feat: drop down 4 layer

* ams1117
Parts:
- removed J1: 12, TestPoint:TestPoint_THTPad_1.0x1.0mm_Drill0.5mm, symbol Connector:Conn_01x01_Pin
- added C1 (x2): 100nF, Capacitor_SMD:C_0603_1608Metric, symbol Device:C
- J1: footprint TestPoint:TestPoint_THTPad_1.0x1.0mm_Drill0.5mm -> TestPoint:TestPoint_THTPad_1.5x1.5mm_Drill0.7mm
- U1: value AP7381-33Y-13 -> AMS1117-3.3; LCSC (none) -> C347256
Connections:
- net +3.3V: now also C1.1
- net GND: now also C1.2, C1.2
- net VD: now also C1.1
Changed lines of the file:
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@@
   (junction (at 36.83 67.31) (diameter 0) (color 0 0 0 0)
   )
+  (junction (at 91.44 81.28) (diameter 0) (color 0 0 0 0)
+  )
+  (junction (at 127 81.28) (diameter 0) (color 0 0 0 0)
+  )
   (junction (at 118.11 81.28) (diameter 0) (color 0 0 0 0)
   )
+  (junction (at 127 58.42) (diameter 0) (color 0 0 0 0)
+  )
   (junction (at 35.56 49.53) (diameter 0) (color 0 0 0 0)
   )
@@
   (junction (at 69.85 58.42) (diameter 0) (color 0 0 0 0)
   )
+  (junction (at 91.44 58.42) (diameter 0) (color 0 0 0 0)
+  )
   (wire (pts (xy 36.83 49.53) (xy 36.83 50.8))
     (stroke (width 0) (type default))
   )
-  (wire (pts (xy 118.11 81.28) (xy 134.62 81.28))
+  (wire (pts (xy 118.11 81.28) (xy 127 81.28))
+    (stroke (width 0) (type default))
+  )
+  (wire (pts (xy 91.44 66.04) (xy 91.44 81.28))
     (stroke (width 0) (type default))
   )
@@
     (stroke (width 0) (type default))
   )
-  (wire (pts (xy 134.62 58.42) (xy 125.73 58.42))
-    (stroke (width 0) (type default))
-  )
-  (wire (pts (xy 69.85 58.42) (xy 101.6 58.42))
+  (wire (pts (xy 127 81.28) (xy 134.62 81.28))
+    (stroke (width 0) (type default))
+  )
+  (wire (pts (xy 134.62 58.42) (xy 127 58.42))
+    (stroke (width 0) (type default))
+  )
+  (wire (pts (xy 69.85 58.42) (xy 91.44 58.42))
     (stroke (width 0) (type default))
   )
@@
     (stroke (width 0) (type default))
   )
+  (wire (pts (xy 127 58.42) (xy 125.73 58.42))
+    (stroke (width 0) (type default))
+  )
   (wire (pts (xy 36.83 67.31) (xy 36.83 66.04))
     (stroke (width 0) (type default))
@@
     (stroke (width 0) (type default))
   )
+  (wire (pts (xy 91.44 58.42) (xy 101.6 58.42))
+    (stroke (width 0) (type default))
+  )
   (wire (pts (xy 35.56 67.31) (xy 36.83 67.31))
     (stroke (width 0) (type default))
   )
-  (wire (pts (xy 24.13 81.28) (xy 101.6 81.28))
+  (wire (pts (xy 24.13 81.28) (xy 91.44 81.28))
     (stroke (width 0) (type default))
   )
@@
     (stroke (width 0) (type default))
   )
+  (wire (pts (xy 127 66.04) (xy 127 81.28))
+    (stroke (width 0) (type default))
+  )
   (wire (pts (xy 110.49 58.42) (xy 101.6 58.42))
     (stroke (width 0) (type default))
@@
     (stroke (width 0) (type default))
   )
+  (wire (pts (xy 91.44 81.28) (xy 101.6 81.28))
+    (stroke (width 0) (type default))
+  )
   (wire (pts (xy 118.11 66.04) (xy 118.11 81.28))
     (stroke (width 0) (type default))
@@
       (effects (font (size 1.27 1.27)))
     )
-    (property "Value" "AP7381-33Y-13" (at 118.11 54.61 0)
+    (property "Value" "AMS1117-3.3" (at 118.11 54.61 0)
       (effects (font (size 1.27 1.27)))
     )
@@
       (effects (font (size 1.27 1.27) italic) hide)
     )
-    (property "Datasheet" "https://datasheet.lcsc.com/lcsc/2304140030_Diodes-Incorporated-AP7381-33Y-13_C460411.pdf" (at 118.11 58.42 0)
+    (property "Datasheet" "http://www.advanced-monolithic.com/pdf/ds1117.pdf" (at 118.11 58.42 0)
+      (effects (font (size 1.27 1.27)) hide)
+    )
+    (property "LCSC" "C347256" (at 118.11 58.42 0)
       (effects (font (size 1.27 1.27)) hide)
     )
@@
       (effects (font (size 1.27 1.27)) hide)
     )
-    (property "Footprint" "TestPoint:TestPoint_THTPad_1.0x1.0mm_Drill0.5mm" (at 30.48 67.31 0)
+    (property "Footprint" "TestPoint:TestPoint_THTPad_1.5x1.5mm_Drill0.7mm" (at 30.48 67.31 0)
       (effects (font (size 1.27 1.27)) hide)
     )
@@
     )
   )
+  (symbol (lib_id "Device:C") (at 127 62.23 0) (unit 1)
+    (in_bom yes) (on_board yes) (dnp no)
+    (property "Reference" "C1" (at 130.81 62.23 0)
+      (effects (font (size 1.27 1.27)) (justify left))
+    )
+    (property "Value" "100nF" (at 130.81 64.77 0)
+      (effects (font (size 1.27 1.27)) (justify left))
+    )
+    (property "Footprint" "Capacitor_SMD:C_0603_1608Metric" (at 127.9652 66.04 0)
+      (effects (font (size 1.27 1.27)) hide)
+    )
+    (property "Datasheet" "~" (at 127 62.23 0)
+      (effects (font (size 1.27 1.27)) hide)
+    )
+    (pin "1")
+    (pin "2")
+    (instances
+      (project "RP2040-Decoder"
+        (path "/11d18738-0f49-4d63-b61c-22a93efd5959"
+          (reference "C1") (unit 1)
+        )
+      )
+      (project "dropdown"
+        (path "/ec2f4957-61c3-483a-b4f9-a4aea502722c"
+          (reference "C4") (unit 1)
+        )
+      )
+    )
+  )
   (symbol (lib_id "Connector:Conn_01x01_Pin") (at 179.07 80.01 90) (unit 1)
     (in_bom yes) (on_board yes) (dnp no)
@@
       (effects (font (size 1.27 1.27)) hide)
     )
-    (property "Footprint" "TestPoint:TestPoint_THTPad_1.0x1.0mm_Drill0.5mm" (at 179.07 80.01 0)
+    (property "Footprint" "TestPoint:TestPoint_THTPad_1.5x1.5mm_Drill0.7mm" (at 179.07 80.01 0)
       (effects (font (size 1.27 1.27)) hide)
     )
@@
     )
   )
-  (symbol (lib_id "Connector:Conn_01x01_Pin") (at 162.56 80.01 270) (mirror x) (unit 1)
-    (in_bom yes) (on_board yes) (dnp no)
-    (property "Reference" "J1" (at 162.56 81.28 0)
-      (effects (font (size 1.27 1.27)))
-    )
-    (property "Value" "12" (at 162.56 85.09 0)
-      (effects (font (size 1.27 1.27)) hide)
-    )
-    (property "Footprint" "TestPoint:TestPoint_THTPad_1.0x1.0mm_Drill0.5mm" (at 162.56 80.01 0)
-      (effects (font (size 1.27 1.27)) hide)
-    )
-    (property "Datasheet" "~" (at 162.56 80.01 0)
-      (effects (font (size 1.27 1.27)) hide)
-    )
-    (pin "1")
-    (instances
-      (project "RP2040-Decoder"
-        (path "/11d18738-0f49-4d63-b61c-22a93efd5959"
-          (reference "J1") (unit 1)
-        )
-      )
-      (project "dropdown"
-        (path "/ec2f4957-61c3-483a-b4f9-a4aea502722c"
-          (reference "J5") (unit 1)
-        )
-      )
-    )
-  )
   (symbol (lib_id "Connector:Conn_01x01_Pin") (at 171.45 80.01 90) (unit 1)
     (in_bom yes) (on_board yes) (dnp no)
@@
       (effects (font (size 1.27 1.27)) hide)
     )
-    (property "Footprint" "TestPoint:TestPoint_THTPad_1.0x1.0mm_Drill0.5mm" (at 171.45 80.01 0)
+    (property "Footprint" "TestPoint:TestPoint_THTPad_1.5x1.5mm_Drill0.7mm" (at 171.45 80.01 0)
       (effects (font (size 1.27 1.27)) hide)
     )
@@
       (effects (font (size 1.27 1.27)) hide)
     )
-    (property "Footprint" "TestPoint:TestPoint_THTPad_1.0x1.0mm_Drill0.5mm" (at 190.5 80.01 0)
+    (property "Footprint" "TestPoint:TestPoint_THTPad_1.5x1.5mm_Drill0.7mm" (at 190.5 80.01 0)
       (effects (font (size 1.27 1.27)) hide)
     )
@@
       (effects (font (size 1.27 1.27)) hide)
     )
-    (property "Footprint" "TestPoint:TestPoint_THTPad_1.0x1.0mm_Drill0.5mm" (at 205.74 80.01 0)
+    (property "Footprint" "TestPoint:TestPoint_THTPad_1.5x1.5mm_Drill0.7mm" (at 205.74 80.01 0)
       (effects (font (size 1.27 1.27)) hide)
     )
@@
       (effects (font (size 1.27 1.27)) hide)
     )
-    (property "Footprint" "TestPoint:TestPoint_THTPad_1.0x1.0mm_Drill0.5mm" (at 185.42 78.74 0)
+    (property "Footprint" "TestPoint:TestPoint_THTPad_1.5x1.5mm_Drill0.7mm" (at 185.42 78.74 0)
       (effects (font (size 1.27 1.27)) hide)
     )
@@
     )
   )
+  (symbol (lib_id "Device:C") (at 91.44 62.23 0) (unit 1)
+    (in_bom yes) (on_board yes) (dnp no)
+    (property "Reference" "C1" (at 95.25 62.23 0)
+      (effects (font (size 1.27 1.27)) (justify left))
+    )
+    (property "Value" "100nF" (at 95.25 64.77 0)
+      (effects (font (size 1.27 1.27)) (justify left))
+    )
+    (property "Footprint" "Capacitor_SMD:C_0603_1608Metric" (at 92.4052 66.04 0)
+      (effects (font (size 1.27 1.27)) hide)
+    )
+    (property "Datasheet" "~" (at 91.44 62.23 0)
+      (effects (font (size 1.27 1.27)) hide)
+    )
+    (pin "1")
+    (pin "2")
+    (instances
+      (project "RP2040-Decoder"
+        (path "/11d18738-0f49-4d63-b61c-22a93efd5959"
+          (reference "C1") (unit 1)
+        )
+      )
+      (project "dropdown"
+        (path "/ec2f4957-61c3-483a-b4f9-a4aea502722c"
+          (reference "C3") (unit 1)
+        )
+      )
+    )
+  )
   (symbol (lib_id "Connector:Conn_01x01_Pin") (at 196.85 81.28 270) (mirror x) (unit 1)
     (in_bom yes) (on_board yes) (dnp no)
@@
       (effects (font (size 1.27 1.27)) hide)
     )
-    (property "Footprint" "TestPoint:TestPoint_THTPad_1.0x1.0mm_Drill0.5mm" (at 196.85 81.28 0)
+    (property "Footprint" "TestPoint:TestPoint_THTPad_1.5x1.5mm_Drill0.7mm" (at 196.85 81.28 0)
       (effects (font (size 1.27 1.27)) hide)
     )
@@
       (effects (font (size 1.27 1.27)) hide)
     )
-    (property "Footprint" "TestPoint:TestPoint_THTPad_1.0x1.0mm_Drill0.5mm" (at 154.94 80.01 0)
+    (property "Footprint" "TestPoint:TestPoint_THTPad_1.5x1.5mm_Drill0.7mm" (at 154.94 80.01 0)
       (effects (font (size 1.27 1.27)) hide)
     )
@@
       (effects (font (size 1.27 1.27)) hide)
     )
-    (property "Footprint" "TestPoint:TestPoint_THTPad_1.0x1.0mm_Drill0.5mm" (at 30.48 49.53 0)
+    (property "Footprint" "TestPoint:TestPoint_THTPad_1.5x1.5mm_Drill0.7mm" (at 30.48 49.53 0)
       (effects (font (size 1.27 1.27)) hide)
     )
@@
         )
       )
-    )
-  )
-  (symbol (lib_id "power:VD") (at 162.56 74.93 0) (unit 1)
-    (in_bom yes) (on_board yes) (dnp no) (fields_autoplaced)
-    (property "Reference" "#PWR06" (at 162.56 78.74 0)
-      (effects (font (size 1.27 1.27)) hide)
-    )
-    (property "Value" "VD" (at 162.56 69.85 0)
-      (effects (font (size 1.27 1.27)))
-    )
-    (property "Footprint" "" (at 162.56 74.93 0)
-      (effects (font (size 1.27 1.27)) hide)
-    )
-    (property "Datasheet" "" (at 162.56 74.93 0)
-      (effects (font (size 1.27 1.27)) hide)
-    )
-    (pin "1")
-    (instances
-      (project "dropdown"
-        (path "/ec2f4957-61c3-483a-b4f9-a4aea502722c"
-          (reference "#PWR06") (unit 1)
-        )
-      )

Commit message: fix: apply jlcpcb rules (#18)
Parts:
- removed C1 (x2): 100nF, Capacitor_SMD:C_0603_1608Metric, symbol Device:C
- removed J1: G, TestPoint:TestPoint_THTPad_1.5x1.5mm_Drill0.7mm, symbol Connector:Conn_01x01_Pin
Changed lines of the file:
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@@
   (junction (at 36.83 67.31) (diameter 0) (color 0 0 0 0)
   )
-  (junction (at 91.44 81.28) (diameter 0) (color 0 0 0 0)
-  )
-  (junction (at 127 81.28) (diameter 0) (color 0 0 0 0)
-  )
   (junction (at 118.11 81.28) (diameter 0) (color 0 0 0 0)
   )
-  (junction (at 127 58.42) (diameter 0) (color 0 0 0 0)
-  )
   (junction (at 35.56 49.53) (diameter 0) (color 0 0 0 0)
   )
@@
   (junction (at 69.85 58.42) (diameter 0) (color 0 0 0 0)
   )
-  (junction (at 91.44 58.42) (diameter 0) (color 0 0 0 0)
-  )
   (wire (pts (xy 36.83 49.53) (xy 36.83 50.8))
     (stroke (width 0) (type default))
   )
-  (wire (pts (xy 118.11 81.28) (xy 127 81.28))
-    (stroke (width 0) (type default))
-  )
-  (wire (pts (xy 91.44 66.04) (xy 91.44 81.28))
+  (wire (pts (xy 118.11 81.28) (xy 134.62 81.28))
     (stroke (width 0) (type default))
   )
@@
     (stroke (width 0) (type default))
   )
-  (wire (pts (xy 127 81.28) (xy 134.62 81.28))
-    (stroke (width 0) (type default))
-  )
-  (wire (pts (xy 134.62 58.42) (xy 127 58.42))
-    (stroke (width 0) (type default))
-  )
-  (wire (pts (xy 69.85 58.42) (xy 91.44 58.42))
+  (wire (pts (xy 125.73 58.42) (xy 134.62 58.42))
+    (stroke (width 0) (type default))
+  )
+  (wire (pts (xy 69.85 58.42) (xy 101.6 58.42))
     (stroke (width 0) (type default))
   )
@@
     (stroke (width 0) (type default))
   )
-  (wire (pts (xy 127 58.42) (xy 125.73 58.42))
-    (stroke (width 0) (type default))
-  )
   (wire (pts (xy 36.83 67.31) (xy 36.83 66.04))
     (stroke (width 0) (type default))
@@
     (stroke (width 0) (type default))
   )
-  (wire (pts (xy 91.44 58.42) (xy 101.6 58.42))
-    (stroke (width 0) (type default))
-  )
   (wire (pts (xy 35.56 67.31) (xy 36.83 67.31))
     (stroke (width 0) (type default))
   )
-  (wire (pts (xy 24.13 81.28) (xy 91.44 81.28))
-    (stroke (width 0) (type default))
-  )
   (wire (pts (xy 24.13 58.42) (xy 29.21 58.42))
     (stroke (width 0) (type default))
   )
-  (wire (pts (xy 127 66.04) (xy 127 81.28))
-    (stroke (width 0) (type default))
-  )
   (wire (pts (xy 110.49 58.42) (xy 101.6 58.42))
     (stroke (width 0) (type default))
@@
     (stroke (width 0) (type default))
   )
-  (wire (pts (xy 91.44 81.28) (xy 101.6 81.28))
+  (wire (pts (xy 24.13 81.28) (xy 101.6 81.28))
     (stroke (width 0) (type default))
   )
@@
     )
   )
-  (symbol (lib_id "Device:C") (at 127 62.23 0) (unit 1)
-    (in_bom yes) (on_board yes) (dnp no)
-    (property "Reference" "C1" (at 130.81 62.23 0)
-      (effects (font (size 1.27 1.27)) (justify left))
-    )
-    (property "Value" "100nF" (at 130.81 64.77 0)
-      (effects (font (size 1.27 1.27)) (justify left))
-    )
-    (property "Footprint" "Capacitor_SMD:C_0603_1608Metric" (at 127.9652 66.04 0)
-      (effects (font (size 1.27 1.27)) hide)
-    )
-    (property "Datasheet" "~" (at 127 62.23 0)
-      (effects (font (size 1.27 1.27)) hide)
-    )
-    (pin "1")
-    (pin "2")
-    (instances
-      (project "RP2040-Decoder"
-        (path "/11d18738-0f49-4d63-b61c-22a93efd5959"
-          (reference "C1") (unit 1)
-        )
-      )
-      (project "dropdown"
-        (path "/ec2f4957-61c3-483a-b4f9-a4aea502722c"
-          (reference "C4") (unit 1)
-        )
-      )
-    )
-  )
   (symbol (lib_id "Connector:Conn_01x01_Pin") (at 179.07 80.01 90) (unit 1)
     (in_bom yes) (on_board yes) (dnp no)
@@
     )
   )
-  (symbol (lib_id "power:GND") (at 185.42 73.66 0) (mirror x) (unit 1)
-    (in_bom yes) (on_board yes) (dnp no)
-    (property "Reference" "#PWR07" (at 185.42 67.31 0)
-      (effects (font (size 1.27 1.27)) hide)
-    )
-    (property "Value" "GND" (at 185.42 68.58 0)
-      (effects (font (size 1.27 1.27)))
-    )
-    (property "Footprint" "" (at 185.42 73.66 0)
-      (effects (font (size 1.27 1.27)) hide)
-    )
-    (property "Datasheet" "" (at 185.42 73.66 0)
-      (effects (font (size 1.27 1.27)) hide)
-    )
-    (pin "1")
-    (instances
-      (project "dropdown"
-        (path "/ec2f4957-61c3-483a-b4f9-a4aea502722c"
-          (reference "#PWR07") (unit 1)
-        )
-      )
-    )
-  )
   (symbol (lib_id "power:+3.3V") (at 205.74 74.93 0) (unit 1)
     (in_bom yes) (on_board yes) (dnp no) (fields_autoplaced)
@@
     )
   )
-  (symbol (lib_id "Connector:Conn_01x01_Pin") (at 185.42 78.74 90) (unit 1)
-    (in_bom yes) (on_board yes) (dnp no)
-    (property "Reference" "J1" (at 185.42 80.01 0)
-      (effects (font (size 1.27 1.27)))
-    )
-    (property "Value" "G" (at 185.42 83.82 0)
-      (effects (font (size 1.27 1.27)) hide)
-    )
-    (property "Footprint" "TestPoint:TestPoint_THTPad_1.5x1.5mm_Drill0.7mm" (at 185.42 78.74 0)
-      (effects (font (size 1.27 1.27)) hide)
-    )
-    (property "Datasheet" "~" (at 185.42 78.74 0)
-      (effects (font (size 1.27 1.27)) hide)
-    )
-    (pin "1")
-    (instances
-      (project "RP2040-Decoder"
-        (path "/11d18738-0f49-4d63-b61c-22a93efd5959"
-          (reference "J1") (unit 1)
-        )
-      )
-      (project "dropdown"
-        (path "/ec2f4957-61c3-483a-b4f9-a4aea502722c"
-          (reference "J6") (unit 1)
-        )
-      )
-    )
-  )
   (symbol (lib_id "power:+12V") (at 35.56 49.53 0) (unit 1)
     (in_bom yes) (on_board yes) (dnp no) (fields_autoplaced)
@@
         )
       )
-    )
-  )
-  (symbol (lib_id "Device:C") (at 91.44 62.23 0) (unit 1)
-    (in_bom yes) (on_board yes) (dnp no)
-    (property "Reference" "C1" (at 95.25 62.23 0)
-      (effects (font (size 1.27 1.27)) (justify left))
-    )
-    (property "Value" "100nF" (at 95.25 64.77 0)
-      (effects (font (size 1.27 1.27)) (justify left))
-    )
-    (property "Footprint" "Capacitor_SMD:C_0603_1608Metric" (at 92.4052 66.04 0)
-      (effects (font (size 1.27 1.27)) hide)
-    )
-    (property "Datasheet" "~" (at 91.44 62.23 0)
-      (effects (font (size 1.27 1.27)) hide)
-    )
-    (pin "1")
-    (pin "2")
-    (instances
-      (project "RP2040-Decoder"
-        (path "/11d18738-0f49-4d63-b61c-22a93efd5959"
-          (reference "C1") (unit 1)
-        )
-      )
-      (project "dropdown"
-        (path "/ec2f4957-61c3-483a-b4f9-a4aea502722c"
-          (reference "C3") (unit 1)
-        )
-      )
