File: hardware/ldomotordriver/ldomotordriver.kicad_sch (KiCad schematic)
At the start: 15 parts, among them U1 AMS1117-3.3, U2 DRV8870DDA

Commit message: gnd zones
Parts:
- R1: value 0.2 -> C270629
Changed lines of the file:
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@@
 			)
 		)
-		(property "Value" "0.2"
+		(property "Value" "C270629"
 			(at 140.97 43.1799 0)
 			(effects
