File: hardware/esp32/esp32.kicad_pcb (KiCad board)
At the start: 4 copper layers, 23.5 x 54.5 mm, 42 parts, among them U1 AMS1117-3.3, U2 ESP32-S3-MINI-1-N8, U3 ESD7104MUTAG, U4 BDR6133, U5 TLV75801PDRV

Commit message: TPS629210DRLR
Parts:
- removed C17, C18: 10u, Capacitor_SMD:C_0603_1608Metric
- removed C6: 10uF, Capacitor_SMD:C_0603_1608Metric
- removed R8: 5.1k, Resistor_SMD:R_0603_1608Metric
- removed U5: TLV75801PDRV, Package_SON:WSON-6-1EP_2x2mm_P0.65mm_EP1x1.6mm
- added C2: 10uF, Capacitor_SMD:C_0603_1608Metric, F.Cu at (110.3, 42.2)
- added C5: 22uF, Capacitor_SMD:C_0603_1608Metric, F.Cu at (105.9, 46.6)
- added L1: 2.2uH,50mA, PCM_JLCPCB:L_0805, F.Cu at (104.8, 44.2)
- added R4: 249K, Resistor_SMD:R_0603_1608Metric, F.Cu at (107.0, 38.7)
- added R5: 100K, Resistor_SMD:R_0603_1608Metric, F.Cu at (104.3, 41.5)
- C3: value 100nF -> 10uF
- R6: value 1M -> 52.3K
- R7: value 200k -> 1K
- U1: value AMS1117-3.3 -> TPS629210DRLR; footprint Package_TO_SOT_SMD:SOT-89-3 -> TPS629210DRLR:SOT50P160X60-8N
- moved D2 28.0 mm to (105.2, 49.4), turned to 180 degrees
- moved C7 21.2 mm to (110.3, 45.2), turned to 0 degrees
- moved R7 19.4 mm to (104.4, 46.9), turned to 90 degrees
- moved R6 16.4 mm to (110.3, 40.7), turned to 180 degrees
- moved C3 7.01 mm to (110.3, 43.7), turned to 0 degrees
- moved U4 5.42 mm to (105.6, 30.1)
- moved o2 5.42 mm to (110.0, 27.6)
- moved o1 5.42 mm to (110.0, 32.6)
- moved U1 2.47 mm to (107.3, 41.9), turned to 0 degrees
- moved R2 1.64 mm to (108.2, 50.5)
- moved U3 1.16 mm to (112.0, 48.4)
Connections:
- C3 pad 1: Net-(D1-+) -> /5VUSB
- C7 pad 1: VCC -> /5VUSB
- D1 pad 1: Net-(D1-+) -> /5VUSB
- R6 pad 1: Net-(U5-FB) -> GND
- R6 pad 2: VCC -> Net-(U1-MODE/S-CONF)
- R7 pad 1: GND -> Net-(D2-A)
- R7 pad 2: Net-(U5-FB) -> VCC
- U1 pad 1: GND -> Net-(U1-FB/VSET)
- U1 pad 2: VCC -> Net-(U1-PG)
- U1 pad 3: Net-(D1-+) -> VCC
- U4 pad 3: Net-(D1-+) -> /5VUSB
Routing:
- net Net-(D1-+): track 15.2 -> 0.00 mm, vias 2 -> 0
- net VCC: track 84.1 -> 72.7 mm
- net Net-(U2-IO13): track 14.9 -> 9.56 mm, vias 2 -> 0
- net Net-(U2-IO12): track 14.8 -> 9.44 mm, vias 2 -> 0
- net Net-(U5-FB): track 5.09 -> 0.00 mm
- net GND: track 161.9 -> 157.8 mm, vias 53 -> 45
- net Net-(U1-PG): track 0.00 -> 2.62 mm
- net Net-(U1-FB/VSET): track 0.00 -> 1.87 mm
- net Net-(U1-SW): track 0.00 -> 1.79 mm
- net Net-(U1-MODE/S-CONF): track 0.00 -> 1.71 mm
- net Net-(JUSB1-CC1): track 4.93 -> 6.54 mm
- net /5VUSB: track 40.8 -> 41.8 mm, vias 0 -> 3
- net /USB_N: track 39.0 -> 38.4 mm
Other:
- copper layers 4 -> 2

Commit message: fix DRC
Routing:
- net GND: track 157.8 -> 164.6 mm, vias 45 -> 46
- net /GPIO0: track 4.05 -> 8.20 mm
- net /5VUSB: track 41.8 -> 45.0 mm
- net VCC: track 72.7 -> 74.8 mm
- net /USB_N: track 38.4 -> 39.0 mm
Changed lines of the file:
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@@
+	)
+	(segment
+		(start 110.35 37.85)
+		(end 108.35 37.85)
+		(width 0.25)
+		(layer "F.Cu")
+		(net 1)
 	)
 	(segment
@@
 	)
 	(segment
+		(start 107 37.85)
+		(end 108.35 37.85)
+		(width 0.1524)
+		(layer "F.Cu")
+		(net 1)
+	)
+	(segment
 		(start 117.1 4.65)
 		(end 117.95 4.65)
@@
 	)
 	(segment
+		(start 108 44)
+		(end 108 42.675)
+		(width 0.1524)
+		(layer "F.Cu")
+		(net 1)
+	)
+	(segment
+		(start 104.435 29.3575)
+		(end 104.935 29.3575)
+		(width 0.25)
+		(layer "F.Cu")
+		(net 1)
+	)
+	(segment
 		(start 111.15 4.65)
 		(end 112 4.65)
@@
 	)
 	(segment
-		(start 104.435 29.3575)
-		(end 104.935 29.3575)
-		(width 0.25)
-		(layer "F.Cu")
-		(net 1)
-	)
-	(segment
 		(start 106.835 29.3575)
 		(end 106.335 29.3575)
@@
 	)
 	(segment
+		(start 111.15 40.675)
+		(end 111.15 38.65)
+		(width 0.25)
+		(layer "F.Cu")
+		(net 1)
+	)
+	(segment
 		(start 103.73 31.4625)
 		(end 104.435 30.7575)
@@
 	)
 	(segment
-		(start 108 42.675)
-		(end 108 44)
-		(width 0.25)
-		(layer "F.Cu")
-		(net 1)
-	)
-	(segment
 		(start 103.8 5.7)
 		(end 103.5 6)
@@
 	)
 	(segment
+		(start 111.15 38.65)
+		(end 110.35 37.85)
+		(width 0.25)
+		(layer "F.Cu")
+		(net 1)
+	)
+	(segment
 		(start 112.85 4.65)
 		(end 112.85 5.35)
@@
 	)
 	(segment
+		(start 104.935 29.3575)
+		(end 105.635 30.0575)
+		(width 0.25)
+		(layer "F.Cu")
+		(net 1)
+	)
+	(segment
 		(start 107.35 50.5)
 		(end 107.35 52.065)
@@
 	)
 	(segment
-		(start 104.935 29.3575)
-		(end 105.635 30.0575)
-		(width 0.25)
-		(layer "F.Cu")
-		(net 1)
-	)
-	(segment
 		(start 107.725 56.62)
 		(end 108.18 57.075)
@@
 		(end 112 14.5)
 		(width 0.25)
+		(layer "F.Cu")
+		(net 1)
+	)
+	(segment
+		(start 108.35 37.85)
+		(end 108.5 38)
+		(width 0.1524)
 		(layer "F.Cu")
 		(net 1)
@@
 	)
 	(via
+		(at 108.35 37.85)
+		(size 0.604799)
+		(drill 0.299999)
+		(layers "F.Cu" "B.Cu")
+		(net 1)
+	)
+	(via
+		(at 103.73 34.8525)
+		(size 0.604799)
+		(drill 0.299999)
+		(layers "F.Cu" "B.Cu")
+		(net 1)
+	)
+	(via
 		(at 108 6)
 		(size 0.8)
@@
 	(via
 		(at 118 7)
-		(size 0.8)
-		(drill 0.4)
-		(layers "F.Cu" "B.Cu")
-		(net 1)
-	)
-	(via
-		(at 103.73 34.8525)
 		(size 0.8)
 		(drill 0.4)
@@
 	)
 	(segment
+		(start 103.5 7.5)
+		(end 104.9 7.5)
+		(width 0.25)
+		(layer "F.Cu")
+		(net 4)
+	)
+	(segment
 		(start 103 42)
 		(end 103 37)
@@
 	)
 	(segment
+		(start 114 31.5)
+		(end 115.15 31.5)
+		(width 0.25)
+		(layer "F.Cu")
+		(net 4)
+	)
+	(segment
+		(start 102.5 6.5)
+		(end 103.5 7.5)
+		(width 0.25)
+		(layer "F.Cu")
+		(net 4)
+	)
+	(segment
+		(start 104.4325 46.08)
+		(end 105.7075 46.08)
+		(width 0.25)
+		(layer "F.Cu")
+		(net 4)
+	)
+	(segment
+		(start 110.5 36)
+		(end 111.5 35)
+		(width 0.25)
+		(layer "F.Cu")
+		(net 4)
+	)
+	(segment
 		(start 104.9 7.5)
 		(end 105 7.4)
@@
 	)
 	(segment
-		(start 114 31.5)
-		(end 115.15 31.5)
-		(width 0.25)
-		(layer "F.Cu")
-		(net 4)
-	)
-	(segment
-		(start 103 7.5)
-		(end 104.9 7.5)
-		(width 0.25)
-		(layer "F.Cu")
-		(net 4)
-	)
-	(segment
-		(start 104.4325 46.08)
-		(end 105.7075 46.08)
-		(width 0.25)
-		(layer "F.Cu")
-		(net 4)
-	)
-	(segment
-		(start 110.5 36)
-		(end 111.5 35)
-		(width 0.25)
-		(layer "F.Cu")
-		(net 4)
-	)
-	(segment
 		(start 104.3175 45.965)
 		(end 104.4325 46.08)
@@
 	)
 	(via
-		(at 103 7.5)
+		(at 102.5 6.5)
 		(size 0.8)
 		(drill 0.4)
@@
 	)
 	(segment
+		(start 103 7)
+		(end 102.5 6.5)
+		(width 0.25)
+		(layer "B.Cu")
+		(net 4)
+	)
+	(segment
 		(start 103 24)
-		(end 103 7.5)
+		(end 103 7)
 		(width 0.25)
 		(layer "B.Cu")
@@
 	)
 	(segment
-		(start 103 8.5)
-		(end 104.75 8.5)
-		(width 0.25)
+		(start 105 8.25)
+		(end 103.25 8.25)
+		(width 0.1524)
 		(layer "F.Cu")
 		(net 9)
 	)
 	(segment
-		(start 104.75 8.5)
-		(end 105 8.25)
-		(width 0.25)
+		(start 103.25 8.25)
+		(end 103 8.5)
+		(width 0.1524)
 		(layer "F.Cu")
 		(net 9)
@@
 	)
 	(segment
+		(start 103 12.65)
+		(end 103 8.5)
+		(width 0.25)
+		(layer "F.Cu")
+		(net 9)
+	)
+	(segment
 		(start 109.5 46.5)
 		(end 109.5 45.175)
@@
 	)
 	(segment
+		(start 111.5 47)
+		(end 111 46.5)
+		(width 0.1524)
+		(layer "F.Cu")
+		(net 33)
+	)
+	(segment
 		(start 109.5 42.175)
 		(end 109.5 43.675)
@@
 	)
 	(segment
+		(start 111 46.5)
+		(end 109.5 46.5)
+		(width 0.1524)
+		(layer "F.Cu")
+		(net 33)
+	)
+	(segment
 		(start 110.1 52.894999)
 		(end 110.1 52.32)
@@
 	)
 	(segment
-		(start 111.449 49.52428)
-		(end 111.449 48.7375)
+		(start 111.5 47.9625)
+		(end 111.5 47)
+		(width 0.1524)
+		(layer "F.Cu")
+		(net 33)
+	)
+	(segment
+		(start 111.5 48.7375)
+		(end 111.5 49.47328)
 		(width 0.25)
 		(layer "F.Cu")
@@
 	)
 	(segment
-		(start 112.503907 49.082814)
-		(end 112.503907 48.7375)
-		(width 0.155814)
-		(layer "F.Cu")
-		(net 35)
-	)
-	(segment
 		(start 111.421093 53.226487)
 		(end 111.75 52.89758)
@@
 	)
 	(segment
+		(start 112.75 52.32)
+		(end 112.75 51.745001)
+		(width 0.155814)
+		(layer "F.Cu")
+		(net 35)
+	)
+	(segment
+		(start 112 20)
+		(end 112.5 20.5)
+		(width 0.2)
+		(layer "F.Cu")
+		(net 35)
+	)
+	(segment
+		(start 112.5 51.495001)
+		(end 112.5 48.7375)
+		(width 0.155814)
+		(layer "F.Cu")
+		(net 35)
+	)
+	(segment
+		(start 112.75 51.745001)
+		(end 112.5 51.495001)
+		(width 0.155814)
+		(layer "F.Cu")
+		(net 35)
+	)
+	(segment
 		(start 112 18.65)
 		(end 112 20)
@@
 	)
 	(segment
-		(start 112.75 49.328907)
-		(end 112.503907 49.082814)
+		(start 112.5 47.9625)
+		(end 112.5 20.5)
 		(width 0.155814)
-		(layer "F.Cu")
-		(net 35)
-	)
-	(segment
-		(start 112.75 52.32)
-		(end 112.75 49.328907)
-		(width 0.155814)
-		(layer "F.Cu")
-		(net 35)
-	)
-	(segment
-		(start 112.5 20.5)
-		(end 112.5 47.349)
-		(width 0.2)
 		(layer "F.Cu")
 		(net 35)
@@
 		(end 112.75 54.5)
 		(width 0.155814)
-		(layer "F.Cu")
-		(net 35)
-	)
-	(segment
-		(start 112 20)
-		(end 112.5 20.5)
-		(width 0.2)
 		(layer "F.Cu")
 		(net 35)
@@
 	)
 	(zone
+		(net 1)
+		(net_name "GND")
+		(layer "B.Cu")
+		(hatch edge 0.5)
+		(priority 1)
+		(connect_pads
+			(clearance 0.5)
+		)
+		(min_thickness 0.25)
+		(filled_areas_thickness no)
+		(fill yes
+			(thermal_gap 0.5)
+			(thermal_bridge_width 0.5)
+		)
+		(polygon
+			(pts
+				(xy 100 58) (xy 100 4.5) (xy 122.5 4.5) (xy 122.5 58)
+			)
+		)
+	)
+	(zone

Commit message: jst
Parts:
- removed g1, g2, g3, g4, g5, g6, g7, o1, o10, o2, o3, o4, o5, o6, o7, o8, o9, tr1, tr2: TestPoint, TestPoint:TestPoint_THTPad_1.5x1.5mm_Drill0.7mm
- added J1: Conn_01x02, Connector_JST:JST_SHL_SM02B-SHLS-TF_1x02-1MP_P1.00mm_Horizontal, F.Cu at (120.0, 54.7)
- added J2: Conn_01x02, Connector_JST:JST_SHL_SM02B-SHLS-TF_1x02-1MP_P1.00mm_Horizontal, F.Cu at (109.0, 27.9)
- added J3: Conn_01x02, Connector_JST:JST_SHL_SM02B-SHLS-TF_1x02-1MP_P1.00mm_Horizontal, F.Cu at (102.5, 54.0)
- moved R2 3.25 mm to (107.5, 47.3), turned to 90 degrees
- moved U4 2.57 mm to (103.1, 29.5)
- moved JUSB1 1.29 mm to (111.2, 55.7)
- moved R1 1.17 mm to (115.8, 50.0)
- moved D1 0.78 mm to (119.0, 45.1), turned to -90 degrees
- moved U3 0.50 mm to (112.0, 47.9)
Connections:
- U2 pad 13: Net-(U2-IO9) -> unconnected-(U2-IO9-Pad13)
- U2 pad 14: Net-(U2-IO10) -> unconnected-(U2-IO10-Pad14)
- U2 pad 15: Net-(U2-IO11) -> unconnected-(U2-IO11-Pad15)
- U2 pad 28: Net-(U2-IO33) -> unconnected-(U2-IO33-Pad28)
- U2 pad 29: Net-(U2-IO34) -> unconnected-(U2-IO34-Pad29)
- U2 pad 30: Net-(U2-IO48) -> unconnected-(U2-IO48-Pad30)
- U2 pad 32: Net-(U2-IO36) -> unconnected-(U2-IO36-Pad32)
- U2 pad 35: Net-(U2-IO39) -> unconnected-(U2-IO39-Pad35)
- U2 pad 38: Net-(U2-IO42) -> unconnected-(U2-IO42-Pad38)
- U2 pad 41: Net-(U2-IO45) -> unconnected-(U2-IO45-Pad41)
- U2 pad 44: Net-(U2-IO46) -> unconnected-(U2-IO46-Pad44)
Routing:
- net /5VUSB: track 45.0 -> 62.2 mm
- net Net-(U2-IO34): track 14.3 -> 0.00 mm
- net GND: track 164.6 -> 154.5 mm
- net Net-(U2-IO11): track 7.40 -> 0.00 mm
- net Net-(U2-IO48): track 5.78 -> 0.00 mm
- net Net-(U2-IO10): track 4.64 -> 0.00 mm
- net Net-(J2-Pin_1): track 2.48 -> 6.54 mm
- net Net-(U2-IO9): track 3.96 -> 0.00 mm
- net Net-(J1-Pin_1): track 2.19 -> 5.94 mm
- net Net-(U2-IO46): track 3.10 -> 0.00 mm
- net Net-(U2-IO45): track 3.08 -> 0.00 mm
- net Net-(U2-IO42): track 3.06 -> 0.00 mm
- net Net-(U2-IO39): track 3.04 -> 0.00 mm
- net Net-(U2-IO36): track 3.02 -> 0.00 mm
- net Net-(J1-Pin_2): track 2.19 -> 5.11 mm
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