File: hardware/esp32/esp32.kicad_pcb (KiCad board)
At the start: 2 copper layers, 23.5 x 54.5 mm, 27 parts, among them J1 Conn_01x02, J2 Conn_01x02, J3 Conn_01x02, J4 Conn_01x06, U1 TPS629210DRLR, U2 ESP32-S3-MINI-1-N8, U3 ESD7104MUTAG, U4 BDR6133

Commit message: esp32 wip
Parts:
- removed BOOT1, RESET1: ~, Button_Switch_SMD:SW_SPST_PTS810
- removed C1: 0.1uF, Capacitor_SMD:C_0603_1608Metric
- removed C3, C7: 10uF, Capacitor_SMD:C_0603_1608Metric
- removed C5: 22uF, Capacitor_SMD:C_0603_1608Metric
- removed L1: 2.2uH,50mA, PCM_JLCPCB:L_0805
- removed R3: 10k, Resistor_SMD:R_0603_1608Metric
- removed R5: 100K, Resistor_SMD:R_0603_1608Metric
- removed R6: 52.3K, Resistor_SMD:R_0603_1608Metric
- removed R7: 1K, Resistor_SMD:R_0603_1608Metric
- removed U3: ESD7104MUTAG, Package_DFN_QFN:Diodes_UDFN-10_1.0x2.5mm_P0.5mm
- removed U4: BDR6133, Library:SOIC-8-1EP_3.9x4.9mm_P1.27mm_EP2.41x3.3mm_ThermalVias
- added D4: ESD3.3, Diode_SMD:D_SOD-923, F.Cu at (90.5, 46.2)
- added F1: Polyfuse 1A, Fuse:Fuse_1206_3216Metric, F.Cu at (109.0, 77.1)
- added FB1: BLM21PG220, Inductor_SMD:L_0805_2012Metric, F.Cu at (107.0, 76.6)
- added J5: Conn_01x02, Connector_JST:JST_SHL_SM02B-SHLS-TF_1x02-1MP_P1.00mm_Horizontal, F.Cu at (159.7, 63.5)
- added J6: Conn_01x02, Connector_JST:JST_SHL_SM02B-SHLS-TF_1x02-1MP_P1.00mm_Horizontal, F.Cu at (166.6, 63.5)
- added SW1: RESET, Button_Switch_SMD:SW_SPST_B3U-1000P, F.Cu at (119.5, 52.2)
- added SW2: BOOT, Button_Switch_SMD:SW_SPST_B3U-1000P, F.Cu at (88.0, 46.5)
- C2: value 10uF -> 100n; footprint Capacitor_SMD:C_0603_1608Metric -> Capacitor_SMD:C_0402_1005Metric_Pad0.74x0.62mm_HandSolder
- C4: value 0.1uF -> 1u
- D1: value ABS2 -> 1N5817; footprint Diode_SMD:Diode_Bridge_Diotec_ABS -> Diode_SMD:D_SOD-123
- D2: value LED -> ESD3.3; footprint LED_SMD:LED_0603_1608Metric -> Diode_SMD:D_SOD-923
- J4: value Conn_01x06 -> Conn_01x02; footprint Connector_JST:JST_SHL_SM06B-SHLS-TF_1x06-1MP_P1.00mm_Horizontal -> Connector_JST:JST_SHL_SM02B-SHLS-TF_1x02-1MP_P1.00mm_Horizontal
- R1: value 5.1k -> 5.1K; footprint Resistor_SMD:R_0603_1608Metric -> Resistor_SMD:R_0402_1005Metric
- R2: value 5.1k -> 10K; footprint Resistor_SMD:R_0603_1608Metric -> Resistor_SMD:R_0402_1005Metric
- R4: value 249K -> 5.1K; footprint Resistor_SMD:R_0603_1608Metric -> Resistor_SMD:R_0402_1005Metric
- U1: value TPS629210DRLR -> USBLC6-2SC6; footprint TPS629210DRLR:SOT50P160X60-8N -> Package_TO_SOT_SMD:SOT-23-6
- moved J4 50.6 mm to (139.5, 62.5)
- moved R4 41.2 mm to (117.5, 78.5), turned to 0 degrees
- moved C4 41.1 mm to (117.0, 52.8), turned to -90 degrees
- moved U1 34.7 mm to (114.0, 76.0), turned to 90 degrees
- moved D1 34.5 mm to (105.0, 76.7), turned to 90 degrees
- moved J1 31.3 mm to (106.0, 82.7)
- moved C2 30.6 mm to (114.0, 72.5), turned to 90 degrees
- moved R1 28.8 mm to (111.5, 78.5), turned to 180 degrees
- moved JUSB1 28.7 mm to (114.5, 84.2)
- moved U2 28.5 mm to (113.0, 40.1)
- moved J2 21.2 mm to (108.0, 54.2), turned to 0 degrees
- moved J3 11.2 mm to (106.5, 64.5)
- moved D2 10.7 mm to (115.5, 52.4), turned to 90 degrees
- moved R2 9.53 mm to (116.5, 50.5), turned to 0 degrees
Connections:
- C2 pad 1: /5VUSB -> +5V
- C4 pad 1: /GPIO0 -> /ESP32_EN
- D1 pad 1: /5VUSB -> +5V
- D1 pad 2: GND -> Net-(D1-A)
- D2 pad 2: Net-(D2-A) -> /ESP32_EN
- J1 pad 1: Net-(J1-Pin_1) -> GND
- J1 pad 2: Net-(J1-Pin_2) -> +5V
- J3 pad 1: GND -> Net-(J3-Pin_1)
- J3 pad 2: GND -> Net-(J3-Pin_2)
- J4 pad 1: unconnected-(J4-Pin_1-Pad1) -> Net-(J4-Pin_1)
- J4 pad 2: unconnected-(J4-Pin_2-Pad2) -> Net-(J4-Pin_2)
- JUSB1 pad A4: /5VUSB -> Net-(F1-Pad1)
- JUSB1 pad A5: Net-(JUSB1-CC1) -> /CC1
- JUSB1 pad A6: /USB_P -> /D+
- JUSB1 pad A7: /USB_N -> /D-
- JUSB1 pad A9: /5VUSB -> Net-(F1-Pad1)
- JUSB1 pad B4: /5VUSB -> Net-(F1-Pad1)
- JUSB1 pad B5: Net-(JUSB1-CC2) -> /CC2
- JUSB1 pad B6: /USB_P -> /D+
- JUSB1 pad B7: /USB_N -> /D-
- JUSB1 pad B9: /5VUSB -> Net-(F1-Pad1)
- R1 pad 1: Net-(JUSB1-CC2) -> /CC1
- R2 pad 1: Net-(JUSB1-CC1) -> +3V3
- R2 pad 2: GND -> /ESP32_EN
- R4 pad 1: GND -> /CC2
- R4 pad 2: Net-(U1-FB/VSET) -> GND
- U1 pad 1: Net-(U1-FB/VSET) -> /D-
- U1 pad 2: Net-(U1-PG) -> GND
- U1 pad 3: VCC -> /D+
- U1 pad 4: Net-(U1-SW) -> /USB_D+
- U1 pad 5: GND -> +5V
- U1 pad 6: /5VUSB -> /USB_D-
- U2 pad 13: Net-(U2-IO9) -> unconnected-(U2-IO9-Pad13)
- U2 pad 14: Net-(U2-IO10) -> unconnected-(U2-IO10-Pad14)
- U2 pad 16: unconnected-(U2-IO12-Pad16) -> Net-(J2-Pin_2)
- U2 pad 17: unconnected-(U2-IO13-Pad17) -> Net-(J2-Pin_1)
- U2 pad 18: unconnected-(U2-IO14-Pad18) -> Net-(J4-Pin_2)
- U2 pad 19: unconnected-(U2-IO15-Pad19) -> Net-(J4-Pin_1)
- U2 pad 20: unconnected-(U2-IO16-Pad20) -> Net-(J5-Pin_2)
- U2 pad 23: /USB_N -> /USB_D-
- U2 pad 24: /USB_P -> /USB_D+
- U2 pad 5: unconnected-(U2-IO1-Pad5) -> Net-(J3-Pin_2)
- U2 pad 6: unconnected-(U2-IO2-Pad6) -> Net-(J3-Pin_1)
Routing:
- net /5VUSB: track 55.8 -> 0.00 mm, vias 2 -> 0
- net VCC: track 52.4 -> 0.14 mm, vias 4 -> 0
- net GND: track 141.1 -> 92.8 mm, vias 44 -> 38
- net /USB_N: track 41.0 -> 0.00 mm, vias 2 -> 0
- net /USB_P: track 39.1 -> 0.00 mm, vias 2 -> 0
- net /ESP32_EN: track 26.5 -> 1.12 mm, vias 2 -> 1
- net Net-(F1-Pad1): track 0.00 -> 11.5 mm
- net /GPIO0: track 8.20 -> 0.00 mm
- net /D+: track 0.00 -> 7.93 mm, vias 0 -> 2
- net Net-(JUSB1-CC1): track 6.47 -> 0.00 mm, vias 2 -> 0
- net Net-(J1-Pin_1): track 5.94 -> 0.00 mm
- net Net-(J1-Pin_2): track 5.11 -> 0.00 mm
- net /D-: track 0.00 -> 4.60 mm, vias 0 -> 2
- net Net-(U2-IO9): track 3.31 -> 0.00 mm
- net Net-(JUSB1-CC2): track 3.17 -> 0.00 mm
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- added copper zone on F.Cu, net GND
Other:
- board size 23.5 x 54.5 mm -> 22 x 54.5 mm

Commit message: esp32
Parts:
- removed C2: 100n, Capacitor_SMD:C_0402_1005Metric_Pad0.74x0.62mm_HandSolder
- removed D1: 1N5817, Diode_SMD:D_SOD-123
- removed F1: Polyfuse 1A, Fuse:Fuse_1206_3216Metric
- removed FB1: BLM21PG220, Inductor_SMD:L_0805_2012Metric
- removed J6: Conn_01x02, Connector_JST:JST_SHL_SM02B-SHLS-TF_1x02-1MP_P1.00mm_Horizontal
- removed JUSB1: USB_C_Receptacle_USB2.0, Connector_USB:USB_C_Receptacle_GCT_USB4105-xx-A_16P_TopMnt_Horizontal
- removed R1, R4: 5.1K, Resistor_SMD:R_0402_1005Metric
- removed U1: USBLC6-2SC6, Package_TO_SOT_SMD:SOT-23-6
- added C18: 10u, Capacitor_SMD:C_0603_1608Metric, F.Cu at (103.0, 35.0)
- added TP1: TestPoint, TestPoint:TestPoint_Pad_1.0x1.0mm, F.Cu at (121.0, 57.5)
- added TP2: TestPoint, TestPoint:TestPoint_Pad_1.0x1.0mm, F.Cu at (121.0, 59.5)
- J2: footprint Connector_JST:JST_SHL_SM02B-SHLS-TF_1x02-1MP_P1.00mm_Horizontal -> Connector_JST:JST_ZH_S2B-ZR-SM4A-TF_1x02-1MP_P1.50mm_Horizontal
- moved J5 41.2 mm to (118.5, 62.7)
- moved J1 31.2 mm to (113.2, 52.3)
- moved J4 27.0 mm to (112.5, 62.8)
- moved SW2 15.9 mm to (103.0, 41.2)
- moved D4 15.0 mm to (103.0, 37.9), turned to -90 degrees
- moved D2 4.81 mm to (119.5, 55.1)
- moved J2 2.90 mm to (105.3, 53.1)
- moved C4 2.86 mm to (118.0, 55.5)
- moved J3 1.88 mm to (106.5, 62.7)
- moved R2 1.50 mm to (116.5, 49.0)
- moved SW1 1.00 mm to (119.5, 51.2)
Connections:
- J1 pad 1: GND -> /USB_D-
- J1 pad 2: +5V -> /USB_D+
- J2 pad 1: Net-(J2-Pin_1) -> GND
- J2 pad 2: Net-(J2-Pin_2) -> +3V3
- J5 pad 1: unconnected-(J5-Pin_1-Pad1) -> Net-(J5-Pin_1)
- U2 pad 16: Net-(J2-Pin_2) -> Net-(J3-Pin_1)
- U2 pad 17: Net-(J2-Pin_1) -> Net-(J3-Pin_2)
- U2 pad 18: Net-(J4-Pin_2) -> Net-(J4-Pin_1)
- U2 pad 19: Net-(J4-Pin_1) -> Net-(J4-Pin_2)
- U2 pad 20: Net-(J5-Pin_2) -> Net-(J5-Pin_1)
- U2 pad 21: unconnected-(U2-IO17-Pad21) -> Net-(J5-Pin_2)
- U2 pad 3: VCC -> +3V3
- U2 pad 31: unconnected-(U2-IO35-Pad31) -> Net-(U2-IO35)
- U2 pad 32: unconnected-(U2-IO36-Pad32) -> Net-(U2-IO36)
- U2 pad 5: Net-(J3-Pin_2) -> unconnected-(U2-IO1-Pad5)
- U2 pad 6: Net-(J3-Pin_1) -> unconnected-(U2-IO2-Pad6)
Routing:
- net +3V3: track 0.00 -> 34.1 mm, vias 0 -> 2
- net /ESP32_EN: track 1.12 -> 26.6 mm, vias 1 -> 0
- net Net-(U2-IO36): track 0.00 -> 19.9 mm, vias 0 -> 2
- net Net-(J5-Pin_2): track 0.00 -> 18.2 mm
- net Net-(U2-IO35): track 0.00 -> 18.1 mm, vias 0 -> 2
- net Net-(J5-Pin_1): track 0.00 -> 17.0 mm
- net Net-(J4-Pin_2): track 0.00 -> 15.4 mm
- net Net-(J4-Pin_1): track 0.00 -> 15.3 mm
- net Net-(J3-Pin_2): track 0.00 -> 14.4 mm
- net Net-(J3-Pin_1): track 0.00 -> 14.3 mm
- net Net-(F1-Pad1): track 11.5 -> 0.00 mm
- net /D+: track 7.93 -> 0.00 mm, vias 2 -> 0
- net GND: track 92.8 -> 86.7 mm, vias 38 -> 37
- net /USB_D-: track 0.00 -> 5.02 mm
- net /GPIO0: track 0.00 -> 4.82 mm
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Other:
- board size 22 x 54.5 mm -> 22 x 34.2 mm
