File: hardware/ams1117/ams1117.kicad_pcb (KiCad board)
At the start: 2 copper layers, 17.5 x 35.5 mm, 12 parts, among them J1 Conn_01x02, J2 Conn_01x02, J3 Conn_01x02, J4 Conn_01x02, J5 Conn_01x02, U1 AMS1117-3.3, U4 BDR6133

Commit message: ams1117
Connections:
- J5 pad 1: GND -> VCC
- J5 pad 2: VCC -> GND
Routing:
- net VCC: track 25.4 -> 29.3 mm
- net GND: track 24.6 -> 23.2 mm
Changed lines of the file:
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@@
 		(property ki_fp_filters "Pin* Test*")
 		(sheetname "/")
-		(sheetfile "ldo.kicad_sch")
+		(sheetfile "ams1117.kicad_sch")
 		(attr exclude_from_pos_files)
 		(fp_circle
@@
 		(property ki_fp_filters "SOIC-8-1EP_3.9x4.9mm_P1.27mm_EP2.29x3mm")
 		(sheetname "/")
-		(sheetfile "ldo.kicad_sch")
+		(sheetfile "ams1117.kicad_sch")
 		(attr smd)
 		(fp_line
@@
 		(property ki_fp_filters "Connector*:*_1x??_*")
 		(sheetname "/")
-		(sheetfile "ldo.kicad_sch")
+		(sheetfile "ams1117.kicad_sch")
 		(attr smd)
 		(fp_line
@@
 			(layers "F.Cu" "F.Mask" "F.Paste")
 			(roundrect_rratio 0.25)
-			(net 1 "GND")
+			(net 5 "VCC")
 			(pinfunction "Pin_1")
 			(pintype "passive")
@@
 			(layers "F.Cu" "F.Mask" "F.Paste")
 			(roundrect_rratio 0.25)
-			(net 5 "VCC")
+			(net 1 "GND")
 			(pinfunction "Pin_2")
 			(pintype "passive")
@@
 		(property ki_fp_filters "SOT?223*TabPin2*")
 		(sheetname "/")
-		(sheetfile "ldo.kicad_sch")
+		(sheetfile "ams1117.kicad_sch")
 		(attr smd)
 		(fp_line
@@
 		(property ki_fp_filters "C_*")
 		(sheetname "/")
-		(sheetfile "ldo.kicad_sch")
+		(sheetfile "ams1117.kicad_sch")
 		(attr smd)
 		(fp_line
@@
 		(property ki_fp_filters "Diode*Bridge*Diotec*ABS*")
 		(sheetname "/")
-		(sheetfile "ldo.kicad_sch")
+		(sheetfile "ams1117.kicad_sch")
 		(attr smd)
 		(fp_line
@@
 		(property ki_fp_filters "Connector*:*_1x??_*")
 		(sheetname "/")
-		(sheetfile "ldo.kicad_sch")
+		(sheetfile "ams1117.kicad_sch")
 		(attr smd)
 		(fp_line
@@
 		(property ki_fp_filters "Connector*:*_1x??_*")
 		(sheetname "/")
-		(sheetfile "ldo.kicad_sch")
+		(sheetfile "ams1117.kicad_sch")
 		(attr smd)
 		(fp_line
@@
 		(property ki_fp_filters "Connector*:*_1x??_*")
 		(sheetname "/")
-		(sheetfile "ldo.kicad_sch")
+		(sheetfile "ams1117.kicad_sch")
 		(attr smd)
 		(fp_line
@@
 		(property ki_fp_filters "Connector*:*_1x??_*")
 		(sheetname "/")
-		(sheetfile "ldo.kicad_sch")
+		(sheetfile "ams1117.kicad_sch")
 		(attr smd)
 		(fp_line
@@
 		(property ki_fp_filters "C_*")
 		(sheetname "/")
-		(sheetfile "ldo.kicad_sch")
+		(sheetfile "ams1117.kicad_sch")
 		(attr smd)
 		(fp_line
@@
 		(property ki_fp_filters "C_*")
 		(sheetname "/")
-		(sheetfile "ldo.kicad_sch")
+		(sheetfile "ams1117.kicad_sch")
 		(attr smd)
 		(fp_line
@@
 	)
 	(segment
+		(start 107 64.35)
+		(end 108.35 63)
+		(width 0.1524)
+		(layer "F.Cu")
+		(net 1)
+	)
+	(segment
 		(start 116.6 52.4)
 		(end 116.5 52.5)
@@
 	)
 	(segment
-		(start 103.65 62.5)
-		(end 103 62.5)
-		(width 0.1524)
-		(layer "F.Cu")
-		(net 1)
-	)
-	(segment
 		(start 107.9 54.5)
 		(end 109.4 56)
@@
 	)
 	(segment
-		(start 105.5 64.35)
-		(end 103.65 62.5)
-		(width 0.1524)
-		(layer "F.Cu")
-		(net 1)
-	)
-	(segment
 		(start 116 58)
 		(end 116 56.5)
@@
 	)
 	(via
-		(at 103 62.5)
+		(at 108.35 63)
 		(size 0.604799)
 		(drill 0.299999)
@@
 	)
 	(segment
-		(start 113.1 64.35)
-		(end 113.25 64.5)
+		(start 113.25 64.5)
+		(end 111.220541 62.470541)
 		(width 0.1524)
 		(layer "F.Cu")
@@
 	)
 	(segment
+		(start 106.029459 62.470541)
+		(end 105.5 63)
+		(width 0.1524)
+		(layer "F.Cu")
+		(net 5)
+	)
+	(segment
 		(start 113.25 64.5)
 		(end 114 63.75)
@@
 	)
 	(segment
+		(start 105.5 63)
+		(end 105.5 64.35)
+		(width 0.1524)
+		(layer "F.Cu")
+		(net 5)
+	)
+	(segment
 		(start 116.5 54.5)
 		(end 114.5 56.5)
@@
 	)
 	(segment
-		(start 107 64.35)
-		(end 113.1 64.35)
+		(start 111.220541 62.470541)
+		(end 106.029459 62.470541)
 		(width 0.1524)
 		(layer "F.Cu")

Commit message: esp32
Parts:
- moved J3 0.50 mm to (105.5, 59.0)
Changed lines of the file:
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@@
 	(footprint "Connector_JST:JST_SHL_SM02B-SHLS-TF_1x02-1MP_P1.00mm_Horizontal"
 		(layer "F.Cu")
-		(at 105.05 58.95 90)
+		(at 105.55 58.95 90)
 		(descr "JST SHL series connector, SM02B-SHLS-TF (http://www.jst-mfg.com/product/pdf/eng/eSHL.pdf), generated with kicad-footprint-generator")
 		(tags "connector JST SHL horizontal")
@@
 		)
 		(property "LCSC" "C160402"
-			(at 0 0 0)
-			(layer "F.SilkS")
+			(at 0 0 90)
+			(unlocked yes)
+			(layer "F.Fab")
 			(hide yes)
 			(effects
 				(font
-					(size 1.27 1.27)
+					(size 1 1)
 					(thickness 0.15)
 				)
