File: hardware/ams1117/ams1117.kicad_pcb (KiCad board)
At the start: 2 copper layers, 17.5 x 35.5 mm, 12 parts, among them J1 Conn_01x02, J2 Conn_01x02, J3 Conn_01x02, J4 Conn_01x02, J5 Conn_01x02, U1 AMS1117-3.3, U4 BDR6133

Commit message: power supply track sizes
Parts:
- moved J5 1.00 mm to (105.2, 66.0)
Routing:
- net GND: track 23.2 -> 24.9 mm
- net VCC: track 29.3 -> 30.8 mm
Changed lines of the file:
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@@
 	(footprint "Connector_JST:JST_ZH_S2B-ZR-SM4A-TF_1x02-1MP_P1.50mm_Horizontal"
 		(layer "F.Cu")
-		(at 106.25 66)
+		(at 105.25 66)
 		(descr "JST ZH series connector, S2B-ZR-SM4A-TF (http://www.jst-mfg.com/product/pdf/eng/eZH.pdf), generated with kicad-footprint-generator")
 		(tags "connector JST ZH horizontal")
@@
 	)
 	(segment
-		(start 107.9 51.5)
-		(end 107.9 52)
-		(width 0.25)
+		(start 116 58)
+		(end 116 57.5)
+		(width 0.1524)
 		(layer "F.Cu")
 		(net 1)
 	)
 	(segment
-		(start 107 64.35)
-		(end 108.35 63)
-		(width 0.1524)
+		(start 107.9 51.5)
+		(end 107.9 52)
+		(width 0.25)
 		(layer "F.Cu")
 		(net 1)
@@
 	)
 	(segment
+		(start 116 57.5)
+		(end 117 56.5)
+		(width 0.5)
+		(layer "F.Cu")
+		(net 1)
+	)
+	(segment
 		(start 107.9 54.5)
 		(end 109.4 56)
-		(width 0.25)
+		(width 0.5)
 		(layer "F.Cu")
 		(net 1)
@@
 		(start 116.6 50.95)
 		(end 116.6 52.4)
-		(width 0.25)
+		(width 0.5)
 		(layer "F.Cu")
 		(net 1)
@@
 		(start 109.675 54.605)
 		(end 109.675 55.725)
-		(width 0.25)
+		(width 0.5)
 		(layer "F.Cu")
 		(net 1)
@@
 		(start 114.875 52.5)
 		(end 114.875 54)
-		(width 0.25)
+		(width 0.5)
 		(layer "F.Cu")
 		(net 1)
@@
 		(start 116.5 52.5)
 		(end 114.875 52.5)
-		(width 0.25)
+		(width 0.5)
 		(layer "F.Cu")
 		(net 1)
 	)
 	(segment
-		(start 116 58)
-		(end 116 56.5)
+		(start 106 64.35)
+		(end 106.35 64)
 		(width 0.1524)
 		(layer "F.Cu")
@@
 		(start 114.875 54)
 		(end 114.875 55.125)
-		(width 0.25)
+		(width 0.5)
 		(layer "F.Cu")
 		(net 1)
@@
 		(start 114.75 64.5)
 		(end 116.25 63)
-		(width 0.1524)
+		(width 0.5)
 		(layer "F.Cu")
 		(net 1)
@@
 	)
 	(segment
+		(start 106.35 64)
+		(end 109 64)
+		(width 0.5)
+		(layer "F.Cu")
+		(net 1)
+	)
+	(segment
 		(start 107.2 53.2)
 		(end 106.5 53.9)
@@
 		(start 107.9 53.9)
 		(end 107.9 54.5)
-		(width 0.25)
+		(width 0.5)
 		(layer "F.Cu")
 		(net 1)
@@
 	)
 	(via
-		(at 116 56.5)
+		(at 109 64)
 		(size 0.604799)
 		(drill 0.299999)
@@
 	)
 	(via
-		(at 108.35 63)
+		(at 117 56.5)
 		(size 0.604799)
 		(drill 0.299999)
@@
 		(start 113.325 52.5)
 		(end 113.325 54)
-		(width 0.25)
+		(width 0.5)
 		(layer "F.Cu")
 		(net 2)
@@
 		(start 111.485 52.065)
 		(end 112.6 50.95)
-		(width 0.1524)
+		(width 0.5)
 		(layer "F.Cu")
 		(net 2)
@@
 		(start 109.675 52.065)
 		(end 111.485 52.065)
-		(width 0.1524)
+		(width 0.5)
 		(layer "F.Cu")
 		(net 2)
@@
 		(start 112.6 51.775)
 		(end 113.325 52.5)
-		(width 0.25)
+		(width 0.5)
 		(layer "F.Cu")
 		(net 2)
@@
 		(start 112.6 50.95)
 		(end 112.6 51.775)
-		(width 0.25)
+		(width 0.5)
 		(layer "F.Cu")
 		(net 2)
@@
 		(start 113.325 54)
 		(end 113.325 57.675)
-		(width 0.25)
+		(width 0.5)
 		(layer "F.Cu")
 		(net 2)
@@
 		(start 112.6 45)
 		(end 112.6 42.55)
-		(width 0.1524)
+		(width 0.5)
 		(layer "F.Cu")
 		(net 3)
@@
 		(start 116.6 44.35)
 		(end 114.45 42.2)
-		(width 0.1524)
+		(width 0.5)
 		(layer "F.Cu")
 		(net 4)
@@
 		(start 116.6 45)
 		(end 116.6 44.35)
-		(width 0.1524)
+		(width 0.5)
 		(layer "F.Cu")
 		(net 4)
 	)
 	(segment
+		(start 113.25 64.5)
+		(end 111.220541 62.470541)
+		(width 0.5)
+		(layer "F.Cu")
+		(net 5)
+	)
+	(segment
 		(start 109.675 53.335)
 		(end 111.335 53.335)
-		(width 0.1524)
+		(width 0.5)
 		(layer "F.Cu")
 		(net 5)
 	)
 	(segment
-		(start 113.25 64.5)
-		(end 111.220541 62.470541)
-		(width 0.1524)
+		(start 114.5 56.5)
+		(end 115.5 56.5)
+		(width 0.5)
 		(layer "F.Cu")
 		(net 5)
 	)
 	(segment
-		(start 114 63.75)
-		(end 114 58.5875)
-		(width 0.1524)
+		(start 105.029459 62.470541)
+		(end 104.5 63)
+		(width 0.5)
 		(layer "F.Cu")
 		(net 5)
 	)
 	(segment
-		(start 106.029459 62.470541)
-		(end 105.5 63)
-		(width 0.1524)
+		(start 104.5 63)
+		(end 104.5 64.35)
+		(width 0.5)
 		(layer "F.Cu")
 		(net 5)
 	)
 	(segment
-		(start 113.25 64.5)
-		(end 114 63.75)
-		(width 0.1524)
+		(start 116.5 55.5)
+		(end 116.5 54.05)
+		(width 0.5)
 		(layer "F.Cu")
 		(net 5)
 	)
 	(segment
-		(start 105.5 63)
-		(end 105.5 64.35)
-		(width 0.1524)
+		(start 114 63.75)
+		(end 114 58.5875)
+		(width 0.5)
 		(layer "F.Cu")
 		(net 5)
 	)
 	(segment
-		(start 116.5 54.5)
-		(end 114.5 56.5)
-		(width 0.1524)
+		(start 111.220541 62.470541)
+		(end 105.029459 62.470541)
+		(width 0.5)
 		(layer "F.Cu")
 		(net 5)
 	)
 	(segment
-		(start 116.5 54.05)
-		(end 116.5 54.5)
-		(width 0.1524)
+		(start 113.25 64.5)
+		(end 114 63.75)
+		(width 0.5)
 		(layer "F.Cu")
 		(net 5)
 	)
 	(segment
-		(start 114.5 56.5)
-		(end 114.5 58.0875)
-		(width 0.1524)
+		(start 115.5 56.5)
+		(end 116.5 55.5)
+		(width 0.5)
 		(layer "F.Cu")
 		(net 5)
 	)
 	(segment
-		(start 114 58.5875)
+		(start 114.5 56.5)
 		(end 114.5 58.0875)
-		(width 0.1524)
+		(width 0.5)
 		(layer "F.Cu")
 		(net 5)
 	)
 	(segment
-		(start 111.220541 62.470541)
-		(end 106.029459 62.470541)
-		(width 0.1524)
+		(start 114 58.5875)
+		(end 114.5 58.0875)
+		(width 0.5)
 		(layer "F.Cu")
 		(net 5)
@@
 		(start 111.335 53.335)
 		(end 111.335 55.335)
-		(width 0.1524)
+		(width 0.5)
 		(layer "B.Cu")
 		(net 5)
@@
 		(start 112.5 56.5)
 		(end 114.5 56.5)
-		(width 0.1524)
+		(width 0.5)
 		(layer "B.Cu")
 		(net 5)
@@
 		(start 112 56)
 		(end 112.5 56.5)
-		(width 0.1524)
+		(width 0.5)
 		(layer "B.Cu")
 		(net 5)
@@
 		(start 111.335 55.335)
 		(end 112 56)
-		(width 0.1524)
+		(width 0.5)
 		(layer "B.Cu")
 		(net 5)
@@
 		(start 109.545 50.795)
 		(end 106.45 47.7)
-		(width 0.1524)
+		(width 0.5)
 		(layer "F.Cu")
 		(net 6)
@@
 		(start 104.725 50.795)
 		(end 104.725 47.925)
-		(width 0.1524)
+		(width 0.5)
 		(layer "F.Cu")
 		(net 7)
@@
 		(start 103.375 59.45)
 		(end 102.45 59.45)
-		(width 0.1524)
+		(width 0.3)
 		(layer "F.Cu")
 		(net 9)
@@
 		(start 102.45 59.45)
 		(end 101.5 58.5)
-		(width 0.1524)
+		(width 0.3)
 		(layer "F.Cu")
 		(net 9)
@@
 		(start 101.5 58.5)
 		(end 101.5 54.315001)
-		(width 0.1524)
+		(width 0.3)
 		(layer "F.Cu")
 		(net 9)
@@
 		(start 101.5 54.315001)
 		(end 103.750001 52.065)
-		(width 0.1524)
+		(width 0.3)
 		(layer "F.Cu")
 		(net 9)
@@
 		(start 103.750001 52.065)
 		(end 104.725 52.065)
-		(width 0.1524)
+		(width 0.3)
 		(layer "F.Cu")
 		(net 9)
@@
 		(start 104.725 53.335)
 		(end 103.750001 53.335)
-		(width 0.1524)
+		(width 0.3)
 		(layer "F.Cu")
 		(net 10)
@@
 		(start 103.375 53.710001)
 		(end 103.375 58.45)
-		(width 0.1524)
+		(width 0.3)
 		(layer "F.Cu")
 		(net 10)
@@
 		(start 103.750001 53.335)
 		(end 103.375 53.710001)
-		(width 0.1524)
+		(width 0.3)
 		(layer "F.Cu")
 		(net 10)

Commit message: adjustments
Parts:
- added TP2: TestPoint, TestPoint:TestPoint_Pad_1.0x1.0mm, F.Cu at (104.5, 38.0)
- added TP3: TestPoint, TestPoint:TestPoint_Pad_1.0x1.0mm, F.Cu at (106.5, 38.0)
- added TP4: TestPoint, TestPoint:TestPoint_Pad_1.0x1.0mm, F.Cu at (108.5, 38.0)
- TP1: footprint MountingHole:MountingHole_2.1mm -> TestPoint:TestPoint_Pad_1.0x1.0mm
- moved TP1 2.06 mm to (102.5, 38.0)
Routing:
- net GND: track 24.9 -> 32.9 mm, vias 6 -> 7

Commit message: jlcpcb wip
Parts:
- removed TP1, TP2, TP3, TP4: TestPoint, TestPoint:TestPoint_Pad_1.0x1.0mm
- added J6: Conn_01x01, Connector_PinHeader_1.00mm:PinHeader_1x01_P1.00mm_Vertical, F.Cu at (102.5, 38.0)
- added J7: Conn_01x01, Connector_PinHeader_1.00mm:PinHeader_1x01_P1.00mm_Vertical, F.Cu at (105.0, 38.0)
- added J8: Conn_01x01, Connector_PinHeader_1.00mm:PinHeader_1x01_P1.00mm_Vertical, F.Cu at (107.5, 38.0)
Routing:
- net GND: track 32.9 -> 31.9 mm

Commit message: replace connectors
Parts:
- J1, J2, J4, J5: footprint Connector_JST:JST_ZH_S2B-ZR-SM4A-TF_1x02-1MP_P1.50mm_Horizontal -> LIB_S2B-ZR_LF__SN_:S2BZRLFSN
- moved J2 9.83 mm to (104.2, 64.9)
- moved J5 8.08 mm to (113.2, 64.9)
- moved J1 1.61 mm to (115.0, 41.5)
- moved J4 1.14 mm to (106.8, 45.6)
Routing:
- net Net-(J4-Pin_2): track 3.19 -> 5.41 mm
- net Net-(J4-Pin_1): track 4.51 -> 6.54 mm
- net VCC: track 30.8 -> 32.3 mm
- net Net-(J1-Pin_2): track 2.94 -> 3.87 mm
