File: hardware/ams1117/ams1117.kicad_sch (KiCad schematic)
At the start: 12 parts, among them J1 Conn_01x02, J2 Conn_01x02, J3 Conn_01x02, J4 Conn_01x02, J5 Conn_01x02, U1 AMS1117-3.3, U4 BDR6133

Commit message: ams1117
Connections:
- net GND: now also J5.2 (Pin_2); no longer J5.1 (Pin_1)
- net VCC: now also J5.1 (Pin_1); no longer J5.2 (Pin_2)
Other:
- moved on the sheet: J5
Changed lines of the file:
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@@
 		(color 0 0 0 0)
 	)
-	(junction
-		(at 101.6 54.61)
-		(diameter 0)
-		(color 0 0 0 0)
-	)
 	(wire
 		(pts
@@
 	(wire
 		(pts
-			(xy 115.57 54.61) (xy 101.6 54.61)
-		)
-		(stroke
-			(width 0)
-			(type default)
-		)
-	)
-	(wire
-		(pts
 			(xy 20.32 68.58) (xy 44.45 68.58)
 		)
@@
 	(wire
 		(pts
-			(xy 115.57 41.91) (xy 115.57 54.61)
-		)
-		(stroke
-			(width 0)
-			(type default)
-		)
-	)
-	(wire
-		(pts
-			(xy 101.6 39.37) (xy 115.57 39.37)
-		)
-		(stroke
-			(width 0)
-			(type default)
-		)
-	)
-	(wire
-		(pts
 			(xy 153.67 33.02) (xy 140.97 33.02)
 		)
@@
 	(wire
 		(pts
-			(xy 153.67 40.64) (xy 144.78 40.64)
-		)
-		(stroke
-			(width 0)
-			(type default)
-		)
-	)
-	(wire
-		(pts
 			(xy 64.77 54.61) (xy 72.39 54.61)
 		)
@@
 			(width 0)
 			(type default)
+		)
+	)
+	(symbol
+		(lib_id "power:GND")
+		(at 115.57 41.91 270)
+		(unit 1)
+		(exclude_from_sim no)
+		(in_bom yes)
+		(on_board yes)
+		(dnp no)
+		(fields_autoplaced yes)
+		(property "Reference" "#PWR09"
+			(at 109.22 41.91 0)
+			(effects
+				(font
+					(size 1.27 1.27)
+				)
+				(hide yes)
+			)
+		)
+		(property "Value" "GND"
+			(at 111.76 41.9099 90)
+			(effects
+				(font
+					(size 1.27 1.27)
+				)
+				(justify right)
+			)
+		)
+		(property "Footprint" ""
+			(at 115.57 41.91 0)
+			(effects
+				(font
+					(size 1.27 1.27)
+				)
+				(hide yes)
+			)
+		)
+		(property "Datasheet" ""
+			(at 115.57 41.91 0)
+			(effects
+				(font
+					(size 1.27 1.27)
+				)
+				(hide yes)
+			)
+		)
+		(property "Description" "Power symbol creates a global label with name \"GND\" , ground"
+			(at 115.57 41.91 0)
+			(effects
+				(font
+					(size 1.27 1.27)
+				)
+				(hide yes)
+			)
+		)
+		(pin "1"
+		)
+		(instances
+			(project "ams1117"
+				(path "/9d64b1b8-57eb-4218-8a7c-add3e4ef813a"
+					(reference "#PWR09")
+					(unit 1)
+				)
+			)
 		)
 	)
@@
 	)
 	(symbol
+		(lib_id "power:VCC")
+		(at 115.57 39.37 90)
+		(unit 1)
+		(exclude_from_sim no)
+		(in_bom yes)
+		(on_board yes)
+		(dnp no)
+		(fields_autoplaced yes)
+		(property "Reference" "#PWR07"
+			(at 119.38 39.37 0)
+			(effects
+				(font
+					(size 1.27 1.27)
+				)
+				(hide yes)
+			)
+		)
+		(property "Value" "VCC"
+			(at 114.3 36.83 90)
+			(effects
+				(font
+					(size 1.27 1.27)
+				)
+			)
+		)
+		(property "Footprint" ""
+			(at 115.57 39.37 0)
+			(effects
+				(font
+					(size 1.27 1.27)
+				)
+				(hide yes)
+			)
+		)
+		(property "Datasheet" ""
+			(at 115.57 39.37 0)
+			(effects
+				(font
+					(size 1.27 1.27)
+				)
+				(hide yes)
+			)
+		)
+		(property "Description" "Power symbol creates a global label with name \"VCC\""
+			(at 115.57 39.37 0)
+			(effects
+				(font
+					(size 1.27 1.27)
+				)
+				(hide yes)
+			)
+		)
+		(pin "1"
+		)
+		(instances
+			(project "ams1117"
+				(path "/9d64b1b8-57eb-4218-8a7c-add3e4ef813a"
+					(reference "#PWR07")
+					(unit 1)
+				)
+			)
+		)
+	)
+	(symbol
 		(lib_id "Device:C")
 		(at 72.39 43.18 0)
@@
 	(symbol
 		(lib_id "Connector_Generic:Conn_01x02")
-		(at 158.75 38.1 0)
+		(at 120.65 31.75 0)
 		(unit 1)
 		(exclude_from_sim no)
@@
 		(fields_autoplaced yes)
 		(property "Reference" "J5"
-			(at 161.29 38.0999 0)
+			(at 123.19 31.7499 0)
 			(effects
 				(font
@@
 		)
 		(property "Value" "Conn_01x02"
-			(at 161.29 40.6399 0)
+			(at 123.19 34.2899 0)
 			(effects
 				(font
@@
 		)
 		(property "Footprint" "Connector_JST:JST_ZH_S2B-ZR-SM4A-TF_1x02-1MP_P1.50mm_Horizontal"
-			(at 158.75 38.1 0)
+			(at 120.65 31.75 0)
 			(effects
 				(font
@@
 		)
 		(property "Datasheet" "~"
-			(at 158.75 38.1 0)
+			(at 120.65 31.75 0)
 			(effects
 				(font
@@
 		)
 		(property "Description" "Generic connector, single row, 01x02, script generated (kicad-library-utils/schlib/autogen/connector/)"
-			(at 158.75 38.1 0)
+			(at 120.65 31.75 0)
 			(effects
 				(font
@@
 		)
 		(property "LCSC" "C157930"
-			(at 158.75 38.1 0)
+			(at 120.65 31.75 0)
 			(effects
 				(font
@@
 	(symbol
 		(lib_id "power:VCC")
-		(at 144.78 40.64 180)
+		(at 115.57 31.75 90)
 		(unit 1)
 		(exclude_from_sim no)
@@
 		(fields_autoplaced yes)
 		(property "Reference" "#PWR06"
-			(at 144.78 36.83 0)
+			(at 119.38 31.75 0)
 			(effects
 				(font
@@
 		)
 		(property "Value" "VCC"
-			(at 144.78 45.72 0)
+			(at 114.3 29.21 90)
 			(effects
 				(font
@@
 		)
 		(property "Footprint" ""
-			(at 144.78 40.64 0)
+			(at 115.57 31.75 0)
 			(effects
 				(font
@@
 		)
 		(property "Datasheet" ""
-			(at 144.78 40.64 0)
+			(at 115.57 31.75 0)
 			(effects
 				(font
@@
 		)
 		(property "Description" "Power symbol creates a global label with name \"VCC\""
-			(at 144.78 40.64 0)
+			(at 115.57 31.75 0)
 			(effects
 				(font
@@
 	(symbol
 		(lib_id "power:GND")
-		(at 153.67 38.1 270)
+		(at 115.57 34.29 270)
 		(unit 1)
 		(exclude_from_sim no)
@@
 		(fields_autoplaced yes)
 		(property "Reference" "#PWR08"
-			(at 147.32 38.1 0)
+			(at 109.22 34.29 0)
 			(effects
 				(font
@@
 		)
 		(property "Value" "GND"
-			(at 149.86 38.0999 90)
+			(at 111.76 34.2899 90)
 			(effects
 				(font
@@
 		)
 		(property "Footprint" ""
-			(at 153.67 38.1 0)
+			(at 115.57 34.29 0)
 			(effects
 				(font
@@
 		)
 		(property "Datasheet" ""
-			(at 153.67 38.1 0)
+			(at 115.57 34.29 0)
 			(effects
 				(font
@@
 		)
 		(property "Description" "Power symbol creates a global label with name \"GND\" , ground"
-			(at 153.67 38.1 0)
-			(effects
-				(font
+			(at 115.57 34.29 0)
+			(effects
+				(font

Commit message: esp32
Other:
- moved on the sheet: TP1

Commit message: adjustments
Parts:
- added TP2, TP3, TP4: TestPoint, TestPoint:TestPoint_Pad_1.0x1.0mm, symbol Connector:TestPoint
- TP1: footprint MountingHole:MountingHole_2.1mm -> TestPoint:TestPoint_Pad_1.0x1.0mm
Connections:
- net GND: now also TP1.1, TP2.1, TP3.1, TP4.1

Commit message: jlcpcb wip
Parts:
- removed TP1, TP2, TP3, TP4: TestPoint, TestPoint:TestPoint_Pad_1.0x1.0mm, symbol Connector:TestPoint
- added J6, J7, J8: Conn_01x01, Connector_PinHeader_1.00mm:PinHeader_1x01_P1.00mm_Vertical, symbol Connector_Generic:Conn_01x01
Connections:
- net GND: now also J6.1 (Pin_1), J7.1 (Pin_1), J8.1 (Pin_1)

Commit message: replace connectors
Parts:
- J1, J2, J4, J5: footprint Connector_JST:JST_ZH_S2B-ZR-SM4A-TF_1x02-1MP_P1.50mm_Horizontal -> LIB_S2B-ZR_LF__SN_:S2BZRLFSN
