File: hardware/usb/usb.kicad_pcb (KiCad board)
At the start: 2 copper layers, 31.5 x 25.6 mm, 15 parts, among them J1 Conn_01x02, J2 Conn_01x02, J5 Conn_01x02, U1 USBLC6-2SC6, U2 AMS1117-3.3

Commit message: esp32
Parts:
- removed J1: Conn_01x02, Connector_JST:JST_ZH_S2B-ZR-SM4A-TF_1x02-1MP_P1.50mm_Horizontal
- added J3: Conn_01x02, Connector_JST:JST_SHL_SM02B-SHLS-TF_1x02-1MP_P1.00mm_Horizontal, F.Cu at (113.5, 66.0)
Routing:
- net Net-(J3-Pin_1): track 7.05 -> 7.65 mm
