File: hardware/tlc5940/tlc5940.kicad_pcb (KiCad board)
At the start: 2 copper layers, 20.5 x 26 mm, 21 parts, among them J1 Conn_01x06, J5 Conn_01x02, U1 TLC5940PWP

Commit message: jlcpcb wip
Parts:
- removed TP1, TP10, TP11, TP12, TP13, TP14, TP15, TP16, TP2, TP3, TP4, TP5, TP6, TP7, TP8, TP9: TestPoint, TestPoint:TestPoint_Pad_1.0x1.0mm
- added J10: Conn_01x01, Connector_PinHeader_1.00mm:PinHeader_1x01_P1.00mm_Vertical, F.Cu at (108.0, 77.5)
- added J11: Conn_01x01, Connector_PinHeader_1.00mm:PinHeader_1x01_P1.00mm_Vertical, F.Cu at (112.0, 77.5)
- added J12: Conn_01x01, Connector_PinHeader_1.00mm:PinHeader_1x01_P1.00mm_Vertical, F.Cu at (114.5, 77.5)
- added J13: Conn_01x01, Connector_PinHeader_1.00mm:PinHeader_1x01_P1.00mm_Vertical, F.Cu at (117.0, 77.5)
- added J14: Conn_01x01, Connector_PinHeader_1.00mm:PinHeader_1x01_P1.00mm_Vertical, F.Cu at (117.0, 75.0)
- added J15: Conn_01x01, Connector_PinHeader_1.00mm:PinHeader_1x01_P1.00mm_Vertical, F.Cu at (117.0, 73.0)
- added J16: Conn_01x01, Connector_PinHeader_1.00mm:PinHeader_1x01_P1.00mm_Vertical, F.Cu at (117.0, 71.0)
- added J17: Conn_01x01, Connector_PinHeader_1.00mm:PinHeader_1x01_P1.00mm_Vertical, F.Cu at (117.0, 69.0)
- added J18: Conn_01x01, Connector_PinHeader_1.00mm:PinHeader_1x01_P1.00mm_Vertical, F.Cu at (117.0, 67.0)
- added J2: Conn_01x01, Connector_PinHeader_1.00mm:PinHeader_1x01_P1.00mm_Vertical, F.Cu at (100.5, 71.5)
- added J3: Conn_01x01, Connector_PinHeader_1.00mm:PinHeader_1x01_P1.00mm_Vertical, F.Cu at (100.5, 73.5)
- added J4: Conn_01x01, Connector_PinHeader_1.00mm:PinHeader_1x01_P1.00mm_Vertical, F.Cu at (100.5, 75.5)
- added J6: Conn_01x01, Connector_PinHeader_1.00mm:PinHeader_1x01_P1.00mm_Vertical, F.Cu at (100.5, 69.5)
- added J7: Conn_01x01, Connector_PinHeader_1.00mm:PinHeader_1x01_P1.00mm_Vertical, F.Cu at (100.5, 77.5)
- added J8: Conn_01x01, Connector_PinHeader_1.00mm:PinHeader_1x01_P1.00mm_Vertical, F.Cu at (103.0, 77.5)
- added J9: Conn_01x01, Connector_PinHeader_1.00mm:PinHeader_1x01_P1.00mm_Vertical, F.Cu at (105.5, 77.5)
- moved R2 0.50 mm to (115.0, 66.0)
Routing:
- net Net-(J10-Pin_1): track 2.53 -> 4.04 mm
- net Net-(J17-Pin_1): track 6.58 -> 5.87 mm
- net Net-(J16-Pin_1): track 6.02 -> 5.31 mm
- net Net-(J18-Pin_1): track 7.14 -> 6.43 mm
- net Net-(U1-IREF): track 3.78 -> 3.28 mm

Commit message: wip
Parts:
- removed J1: Conn_01x06, Connector_JST:JST_SHL_SM06B-SHLS-TF_1x06-1MP_P1.00mm_Horizontal
- added J19: Conn_01x08, Connector_JST:JST_SHL_SM08B-SHLS-TF_1x08-1MP_P1.00mm_Horizontal, F.Cu at (104.5, 58.0)
Routing:
- net Net-(J19-Pin_2): track 26.6 -> 19.7 mm
- net Net-(J19-Pin_3): track 14.3 -> 8.33 mm, vias 2 -> 0
- net Net-(J19-Pin_6): track 16.0 -> 10.6 mm, vias 2 -> 0
- net Net-(J19-Pin_5): track 14.7 -> 9.69 mm, vias 2 -> 0
- net Net-(J19-Pin_4): track 13.4 -> 9.04 mm, vias 2 -> 0
- net Net-(J19-Pin_7): track 13.5 -> 11.8 mm
Other:
- board size 20.5 x 26 mm -> 21 x 26 mm

Commit message: replace connectors
Parts:
- removed J5: Conn_01x02, Connector_JST:JST_ZH_S2B-ZR-SM4A-TF_1x02-1MP_P1.50mm_Horizontal
- added J1: Conn_01x02, LIB_S2B-ZR_LF__SN_:S2BZRLFSN, F.Cu at (115.2, 59.6)
Routing:
- net GND: track 18.3 -> 19.9 mm
- net VCC: track 13.1 -> 13.8 mm
